File: schematics/power-board/power-board.kicad_sch (KiCad schematic)
At the start: 23 parts, among them J1 5V, J2 5V, J3 +12V, J4 +12V, J5 -12V, J6 -12V, J7 GND, J8 Conn_01x01_Socket, J9 5V, Q1 BT151-500R, SW1 SW, U1 USBC Module, U2 TPS5430 Module 5V, U3 TPS5430 Module 12V

Commit message: refactor: fix PCBBox holes dimensions and remake pcb vias with the new components
Parts:
- removed F1: RXEF200 2A, Fuse:Fuse_Bourns_MF-RG300, symbol Device:Polyfuse
- removed F2, F3: RXEF110 1A1, Fuse:Fuse_Bourns_MF-RG300, symbol Device:Polyfuse
- removed J9: 5V, footprints:Connector, symbol Connector:Conn_01x01_Socket
- added F1, F2, F3: Fuse, Fuse:Fuse_Bourns_MF-RHT200, symbol Device:Fuse
- D1: footprint Diode_THT:D_DO-34_SOD68_P7.62mm_Horizontal -> Diode_THT:D_DO-41_SOD81_P10.16mm_Horizontal
- Q1: footprint Package_TO_SOT_THT:TO-92_Inline -> Package_TO_SOT_THT:TO-220-3_Vertical
- R1: footprint Resistor_THT:R_Axial_DIN0204_L3.6mm_D1.6mm_P5.08mm_Horizontal -> Resistor_THT:R_Axial_DIN0207_L6.3mm_D2.5mm_P10.16mm_Horizontal
Connections:
- net +12V: now also F2.2
- net -12V: now also F3.2
- net 5V: now also F1.2
- net at J1.1 (Pin_1): now also F1.1
- net at J3.1 (Pin_1): now also F2.1
- net at J5.1 (Pin_1): now also F3.1
